File: cad/Eagle/Eagle MainPCB/Schulglocke_PCB.sch (EAGLE design)
At the start: 34 parts, among them IC1 SFH6156, IC2 SFH6156, K1 JS-M1-9V-5, Q3 MUN2112T1, Q4 MUN2211T1

Commit message: korekte bauteile
Parts:
- removed CX1, CX2: (no value), rcl:CXXC22B10
- removed D1: (no value), diode:DIODE-SMB
- removed D2, D3: 1N5333, diode:1N5333
- removed J1: (no value), con-amp:MTA03-156
- removed J2: (no value), con-amp:MTA02-156
- removed Q3: MUN2112T1, transistor-pnp:MUN2112T1
- removed Q4: MUN2211T1, transistor-npn:MUN2211T1
- removed SV1: (no value), con-amp-mt:MT6-4
- added C3, C4: (no value), rcl:C-EU102-064X133
- added D4, D5, D6: 1N4004, diode:1N4004
- added JP1: (no value), pinhead:PINHD-1X2
- added JP2: (no value), pinhead:PINHD-1X3
- added JP3: (no value), pinhead:PINHD-1X4
- added Q1, Q2: BSS123, transistor-small-signal:BSS123
Connections:
- net GND: now also JP1.1, JP3.2, Q1.S, Q2.S; no longer J2.1, Q3.C, Q4.E, SV1-3.S
- net N$1: now also C3.1, C4.2, JP2.2; no longer CX1.1, CX2.2, J1.2
- net N$10: now also D5.A, Q2.D; no longer D1.A, Q3.E
- net N$11: now also JP1.2; no longer J2.2
- net N$15: now also Q1.D; no longer Q4.C
- net N$17: now also Q1.G; no longer Q4.B
- net N$2: now also C4.1, JP2.1; no longer CX1.2, J1.1
- net N$22: now also Q2.G; no longer Q3.B
- net N$3: now also C3.2, JP2.3; no longer CX2.1, J1.3
- net N$4: now also D6.A; no longer D3.A
- net N$5: now also D6.C, JP3.1; no longer D3.C, SV1-4.S
- net N$6: now also JP3.3; no longer SV1-2.S
- net N$7: now also JP3.4; no longer SV1-1.S
- net N$9: now also D4.A; no longer D2.A
- net VCC: now also D4.C, D5.C; no longer D1.C, D2.C

Commit message: neue numerierung
Parts:
- removed C4: (no value), rcl:C-EU102-064X133
- added C2: (no value), rcl:C-EU102-064X133
- C1: device rcl:C-EUC1206K -> rcl:CPOL-EU153CLV-0605
- F1: value (none) -> FUSEBLANK_5X20MM; device fuse:TR5 -> fuse:FUSEBLANK_5X20MM
- F2: value SMD100F/33 -> FUSEBLANK_5X20MM; device switch-raychem:SMD100F/33 -> fuse:FUSEBLANK_5X20MM
- JP2: device pinhead:PINHD-1X3 -> pinhead:PINHD-1X4
- JP3: device pinhead:PINHD-1X4 -> pinhead:PINHD-1X3
- R10, R9: value (none) -> P593; device rcl:R-EU_M1206 -> varistor:P593
- R3, R4: value P593 -> (none); device varistor:P593 -> rcl:R-EU_M1206
- renumbered D4 to D1, D5 to D3, D6 to D2, U$1 to M1, U$2 to M2, U$3 to M3
Connections:
- net +5V: now also R5.2; no longer R2.2
- net GND: now also C1.-, JP2.2, LED2.C, R2.2, R3.2, R4.2, R7.2; no longer C1.2, JP3.2, LED1.C, R10.2, R6.2, R8.2, R9.2
- net N$1: now also C2.1, C3.2, JP3.2, R10.2, R9.1; no longer C3.1, C4.2, JP2.2, R3.2, R4.1
- net N$12: now also LED1.A; no longer LED2.A
- net N$13: now also LED2.A, R6.1; no longer LED1.A, R1.1
- net N$14: now also R5.1; no longer R2.1
- net N$16: now also R1.2; no longer R5.2
- net N$17: now also R1.1, R3.1; no longer R5.1, R6.1
- net N$19: now also IC1LED.K, R4.1; no longer IC2LED.K, R10.1
- net N$2: now also C3.1, JP3.1, R10.1; no longer C4.1, JP2.1, R3.1
- net N$22: now also R8.1; no longer R7.1
- net N$24: now also LED1.C, R2.1; no longer LED2.C, R9.1
- net N$3: now also C2.2, JP3.3, R9.2; no longer C3.2, JP2.3, R4.2
- net N$5: now also JP2.1; no longer JP3.1
- net N$6: now also IC2CE.C, JP2.3; no longer IC1CE.C, JP3.3
- net N$7: now also IC2CE.E, JP2.4; no longer IC1CE.E, JP3.4
- net OPT_ISOL: now also IC1LED.A; no longer IC2LED.A
- net RELAY_EN: now also R6.2, R7.1, R8.2; no longer R1.2, R7.2, R8.1
- net VCC: now also C1.+; no longer C1.1
Other:
- moved on the sheet: C3, LED1, LED2, R1, R2, R5, R6, R7, R8

Commit message: before change
Parts:
- removed IC1, IC2: SFH6156, optocoupler:SFH6156
- added OK1: PC817, optocoupler:PC817
Connections:
- net N$19: now also OK1.C; no longer IC1LED.K
- net N$6: now also OK1.COL; no longer IC2CE.C
- net N$7: now also OK1.EMIT; no longer IC2CE.E
- net OPT_ISOL: now also OK1.A; no longer IC1LED.A
Other:
- moved on the sheet: R4

Commit message: leiterplatte plaziert
Parts:
- removed B1: ARDUINO_MEGA_R3FULL, sparkfun eagle:ARDUINO_MEGA_R3FULL
- removed K1: JS-M1-9V-5, relay:JS-M1-9V-5
- removed S1: (no value), switch:255SB
- added B2: ARDUINO_MEGA_R3_CUSTOM_SHIELDFULL, customlib:ARDUINO_MEGA_R3_CUSTOM_SHIELDFULL
- added C5: (no value), rcl:C-EUC1206K
- added REL1: (no value), special:REL-5PIN
- F1, F2: value FUSEBLANK_5X20MM -> (none); device fuse:FUSEBLANK_5X20MM -> special:FUSE2P
Connections:
- removed net N$11: JP1.2, S1.P
- new net N$18: B2.30
- net +3V3: now also B2.3.3V; no longer B1.3.3V
- net +5V: now also B2.5V; no longer B1.5V
- net ARD_MISO: now also B2.50/MISO; no longer B1.50/MISO
- net ARD_MOSI: now also B2.51/MOSI; no longer B1.51/MOSI
- net ARD_SCK: now also B2.52/SCK; no longer B1.52/SCK
- net ARD_SCL: now also B2.SCL; no longer B1.SCL
- net ARD_SDA: now also B2.SDA; no longer B1.SDA
- net ETH_CS: now also B2.28; no longer B1.28
- net GND: now also B2.GND, B2.GND@2, B2.GND@3, C5.2; no longer B1.GND, B1.GND@2, B1.GND@3
- net LCD_BL: now also B2.9; no longer B1.9
- net LCD_CS: now also B2.10; no longer B1.10
- net LCD_DC: now also B2.7; no longer B1.7
- net LCD_RST: now also B2.8; no longer B1.8
- net N$1: now also REL1.C; no longer K12.P
- net N$10: now also REL1.S1; no longer K11.2
- net N$12: now also B2.24; no longer B1.24
- net N$16: now also B2.22, R3.1; no longer B1.22
- net N$17: no longer R3.1
- net N$2: now also REL1.O; no longer K12.O
- net N$3: now also REL1.S; no longer K12.S
- net N$4: now also F1.2A; no longer F2.2
- net N$8: now also F1.1A, F2.1A, JP1.2; no longer F1.1, F2.1, S1.S
- net N$9: now also F2.2A; no longer F1.2
- net OPT_ISOL: now also B2.26; no longer B1.26
- net SD_CS: now also B2.5; no longer B1.5
- net TP_BUSY: now also B2.6; no longer B1.6
- net TP_CS: now also B2.4; no longer B1.4
- net TP_IRQ: now also B2.3; no longer B1.3
- net VCC: now also B2.VIN, C5.1, REL1.S2; no longer B1.VIN, K11.1
Other:
- note added: "2A"
- note removed: "1B"
- moved on the sheet: C1, C2, C3, JP3, R1, R10, R3, R9

Commit message: mit traces noch ohne montagelöcher und ohne anpassung footprints
Parts:
- removed F2: (no value), special:FUSE2P
Connections:
- removed net N$18: B2.30
- removed net N$8: F1.1A, F2.1A, JP1.2
- net N$9: now also F1.1A, JP1.2; no longer F2.2A
- net RELAY_EN: now also B2.30
Changed lines of the file:
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@@
 <part name="REL1" library="special" library_urn="urn:adsk.eagle:library:367" deviceset="REL-5PIN" device="" package3d_urn="urn:adsk.eagle:package:26666/1"/>
 <part name="B2" library="customlib" deviceset="ARDUINO_MEGA_R3_CUSTOM_SHIELD" device="FULL"/>
-<part name="F2" library="special" library_urn="urn:adsk.eagle:library:367" deviceset="FUSE2P" device="" package3d_urn="urn:adsk.eagle:package:26671/1"/>
 <part name="F1" library="special" library_urn="urn:adsk.eagle:library:367" deviceset="FUSE2P" device="" package3d_urn="urn:adsk.eagle:package:26671/1"/>
 <part name="C5" library="rcl" library_urn="urn:adsk.eagle:library:334" deviceset="C-EU" device="C1206K" package3d_urn="urn:adsk.eagle:package:23682/2"/>
@@
 <attribute name="VALUE" x="35.56" y="10.16" size="1.778" layer="96"/>
 </instance>
-<instance part="F2" gate="G$1" x="48.26" y="162.56" smashed="yes">
-<attribute name="NAME" x="46.99" y="164.465" size="1.778" layer="95"/>
-<attribute name="VALUE" x="45.72" y="159.0802" size="1.778" layer="96"/>
-</instance>
 <instance part="F1" gate="G$1" x="101.6" y="172.72" smashed="yes">
 <attribute name="NAME" x="100.33" y="174.625" size="1.778" layer="95"/>
@@
 </segment>
 <segment>
-<wire x1="66.04" y1="162.56" x2="73.66" y2="162.56" width="0.1524" layer="91"/>
 <pinref part="P+1" gate="VCC" pin="VCC"/>
-<wire x1="73.66" y1="162.56" x2="81.28" y2="162.56" width="0.1524" layer="91"/>
+<wire x1="66.04" y1="162.56" x2="81.28" y2="162.56" width="0.1524" layer="91"/>
 <wire x1="81.28" y1="162.56" x2="81.28" y2="165.1" width="0.1524" layer="91"/>
-<wire x1="73.66" y1="160.02" x2="73.66" y2="162.56" width="0.1524" layer="91"/>
-<junction x="73.66" y="162.56"/>
 <pinref part="D1" gate="1" pin="C"/>
 <wire x1="81.28" y1="162.56" x2="81.28" y2="160.02" width="0.1524" layer="91"/>
@@
 <wire x1="10.16" y1="160.02" x2="55.88" y2="160.02" width="0.1524" layer="91"/>
 <wire x1="55.88" y1="160.02" x2="55.88" y2="149.86" width="0.1524" layer="91"/>
-<wire x1="55.88" y1="149.86" x2="73.66" y2="149.86" width="0.1524" layer="91"/>
-<wire x1="73.66" y1="149.86" x2="81.28" y2="149.86" width="0.1524" layer="91"/>
+<wire x1="55.88" y1="149.86" x2="81.28" y2="149.86" width="0.1524" layer="91"/>
 <pinref part="SUPPLY1" gate="GND" pin="GND"/>
 <wire x1="81.28" y1="149.86" x2="81.28" y2="147.32" width="0.1524" layer="91"/>
-<wire x1="73.66" y1="152.4" x2="73.66" y2="149.86" width="0.1524" layer="91"/>
-<junction x="73.66" y="149.86"/>
 <pinref part="JP1" gate="G$1" pin="1"/>
 <wire x1="81.28" y1="152.4" x2="81.28" y2="149.86" width="0.1524" layer="91"/>
@@
 </segment>
 </net>
-<net name="N$8" class="0">
-<segment>
+<net name="N$9" class="0">
+<segment>
+<pinref part="D1" gate="1" pin="A"/>
 <wire x1="96.52" y1="172.72" x2="40.64" y2="172.72" width="0.1524" layer="91"/>
 <wire x1="40.64" y1="172.72" x2="40.64" y2="162.56" width="0.1524" layer="91"/>
-<wire x1="40.64" y1="162.56" x2="43.18" y2="162.56" width="0.1524" layer="91"/>
-<pinref part="F2" gate="G$1" pin="1A"/>
 <pinref part="F1" gate="G$1" pin="1A"/>
 <wire x1="20.32" y1="162.56" x2="20.32" y2="165.1" width="0.1524" layer="91"/>
@@
 <junction x="20.32" y="162.56"/>
 <junction x="40.64" y="162.56"/>
-</segment>
-</net>
-<net name="N$9" class="0">
-<segment>
-<wire x1="53.34" y1="162.56" x2="60.96" y2="162.56" width="0.1524" layer="91"/>
-<pinref part="D1" gate="1" pin="A"/>
-<pinref part="F2" gate="G$1" pin="2A"/>
+<wire x1="60.96" y1="162.56" x2="40.64" y2="162.56" width="0.1524" layer="91"/>
 </segment>
 </net>
@@
 <junction x="152.4" y="137.16"/>
 <label x="137.16" y="137.16" size="1.778" layer="95" rot="R180"/>
+</segment>
+<segment>
+<wire x1="71.12" y1="43.18" x2="63.5" y2="43.18" width="0.1524" layer="91"/>
+<pinref part="B2" gate="B1" pin="30"/>
 <label x="71.12" y="43.18" size="1.778" layer="95"/>
 </segment>
@@
 </segment>
 </net>
-<net name="N$18" class="0">
-<segment>
-<wire x1="71.12" y1="43.18" x2="63.5" y2="43.18" width="0.1524" layer="91"/>
-<pinref part="B2" gate="B1" pin="30"/>
-</segment>
-</net>

Commit message: added drill holes
Parts:
- added U$1, U$2, U$3: MOUNTPOINT3.3MM, customlib:MOUNTPOINT3.3MM
Changed lines of the file:
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@@
 <part name="SUPPLY11" library="supply2" library_urn="urn:adsk.eagle:library:372" deviceset="GND" device=""/>
 <part name="C1" library="rcl" library_urn="urn:adsk.eagle:library:334" deviceset="CPOL-EU" device="153CLV-0605" package3d_urn="urn:adsk.eagle:package:23398/2"/>
+<part name="U$1" library="customlib" deviceset="MOUNTPOINT3.3MM" device=""/>
+<part name="U$2" library="customlib" deviceset="MOUNTPOINT3.3MM" device=""/>
+<part name="U$3" library="customlib" deviceset="MOUNTPOINT3.3MM" device=""/>
 </parts>
 <sheets>
@@
 <attribute name="VALUE" x="173.863" y="157.9626" size="1.778" layer="96"/>
 </instance>
+<instance part="U$1" gate="G$1" x="12.7" y="68.58" smashed="yes"/>
+<instance part="U$2" gate="G$1" x="12.7" y="83.82" smashed="yes"/>
+<instance part="U$3" gate="G$1" x="12.7" y="53.34" smashed="yes"/>
 </instances>
 <busses>
