File: cad/Eagle/Eagle MainPCB/Schulglocke_PCB.sch (EAGLE design)
At the start: 35 parts, among them M1 DS3231SHIELD, M2 EMC28J60SHIELD, M3 WAVESHAREDISPLAY, Q1 BSS123, Q2 BSS123

Commit message: fixed a name
Parts:
- C1: value (none) -> 47uF
- C2, C3: value (none) -> DNP
- C5: value (none) -> 100nF
- F1: value (none) -> 1A F
- R1, R3, R7, R8: value (none) -> 100K
- R2, R4, R6: value (none) -> 330R
- R5: value (none) -> 680R
Other:
- note added: "DNP"
- note added: "Module"
- note added: "PWR_IN"
- note added: "Relay OUT"
- note added: "Schulglocke Michael Schima Viktor Mandlbauer"
- note removed: "Schulglocke Michael Schima Viktor Mandelbauer"
