File: cad/Eagle/Eagle MainPCB/Schulglocke_PCB.brd (EAGLE design)
At the start: 140 x 90 mm, 35 parts, among them M1 DS3231SHIELD, M2 EMC28J60SHIELD, M3 WAVESHAREDISPLAY, Q1 BSS123, Q2 BSS123

Commit message: fixed a name
Parts:
- C1: value (none) -> 47uF
- C2, C3: value (none) -> DNP
- C5: value (none) -> 100nF
- F1: value (none) -> 1A F
- R1, R3, R7, R8: value (none) -> 100K
- R2, R4, R6: value (none) -> 330R
- R5: value (none) -> 680R
Changed lines of the file:
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@@
 <?xml version="1.0" encoding="utf-8"?>
 <!DOCTYPE eagle SYSTEM "eagle.dtd">
-<eagle version="9.5.2">
+<eagle version="9.6.2">
 <drawing>
 <settings>
@@
 </autorouter>
 <elements>
-<element name="C2" library="rcl" library_urn="urn:adsk.eagle:library:334" package="C102-064X133" package3d_urn="urn:adsk.eagle:package:23653/1" value="" x="103.97" y="10.814" smashed="yes" rot="MR90">
+<element name="C2" library="rcl" library_urn="urn:adsk.eagle:library:334" package="C102-064X133" package3d_urn="urn:adsk.eagle:package:23653/1" value="DNP" x="103.97" y="10.814" smashed="yes" rot="MR90">
 <attribute name="NAME" x="107.399" y="4.718" size="1.27" layer="26" ratio="10" rot="MR90"/>
 <attribute name="POPULARITY" value="0" x="-72.56" y="70.504" size="1.778" layer="28" rot="MR90" display="off"/>
@@
 <attribute name="VALUE" x="101.938" y="9.29" size="1.27" layer="28" ratio="10" rot="MR90"/>
 </element>
-<element name="C3" library="rcl" library_urn="urn:adsk.eagle:library:334" package="C102-064X133" package3d_urn="urn:adsk.eagle:package:23653/1" value="" x="111.03" y="8.436" smashed="yes" rot="MR90">
+<element name="C3" library="rcl" library_urn="urn:adsk.eagle:library:334" package="C102-064X133" package3d_urn="urn:adsk.eagle:package:23653/1" value="DNP" x="111.03" y="8.436" smashed="yes" rot="MR90">
 <attribute name="NAME" x="114.459" y="2.34" size="1.27" layer="26" ratio="10" rot="MR90"/>
 <attribute name="POPULARITY" value="0" x="-65.5" y="82.096" size="1.778" layer="28" rot="MR90" display="off"/>
@@
 <attribute name="VALUE" x="131.161" y="19.269" size="1.27" layer="27"/>
 </element>
-<element name="R1" library="rcl" library_urn="urn:adsk.eagle:library:334" package="M1206" package3d_urn="urn:adsk.eagle:package:23566/2" value="" x="35.394" y="18.31" smashed="yes" rot="R90">
+<element name="R1" library="rcl" library_urn="urn:adsk.eagle:library:334" package="M1206" package3d_urn="urn:adsk.eagle:package:23566/2" value="100K" x="35.394" y="18.31" smashed="yes" rot="R90">
 <attribute name="NAME" x="34.124" y="17.04" size="1.27" layer="25" rot="R90"/>
 <attribute name="POPULARITY" value="17" x="222.084" y="50.06" size="1.778" layer="27" rot="R90" display="off"/>
@@
 <attribute name="VALUE" x="123.181" y="8.35" size="1.27" layer="28" ratio="10" rot="MR270"/>
 </element>
-<element name="R2" library="rcl" library_urn="urn:adsk.eagle:library:334" package="M1206" package3d_urn="urn:adsk.eagle:package:23566/2" value="" x="119.568" y="57.688" smashed="yes" rot="R270">
+<element name="R2" library="rcl" library_urn="urn:adsk.eagle:library:334" package="M1206" package3d_urn="urn:adsk.eagle:package:23566/2" value="330R" x="119.568" y="57.688" smashed="yes" rot="R270">
 <attribute name="NAME" x="120.838" y="58.958" size="1.27" layer="25" rot="R270"/>
 <attribute name="POPULARITY" value="17" x="-67.122" y="20.858" size="1.778" layer="27" rot="R270" display="off"/>
@@
 <attribute name="VALUE" x="117.028" y="58.958" size="1.27" layer="27" rot="R270"/>
 </element>
-<element name="R3" library="rcl" library_urn="urn:adsk.eagle:library:334" package="M1206" package3d_urn="urn:adsk.eagle:package:23566/2" value="" x="32.248" y="24.58" smashed="yes" rot="R180">
+<element name="R3" library="rcl" library_urn="urn:adsk.eagle:library:334" package="M1206" package3d_urn="urn:adsk.eagle:package:23566/2" value="100K" x="32.248" y="24.58" smashed="yes" rot="R180">
 <attribute name="NAME" x="33.518" y="23.31" size="1.27" layer="25" rot="R180"/>
 <attribute name="POPULARITY" value="17" x="-9.662" y="211.27" size="1.778" layer="27" rot="R180" display="off"/>
@@
 <attribute name="VALUE" x="33.518" y="27.12" size="1.27" layer="27" rot="R180"/>
 </element>
-<element name="R4" library="rcl" library_urn="urn:adsk.eagle:library:334" package="M1206" package3d_urn="urn:adsk.eagle:package:23566/2" value="" x="25.574" y="24.852" smashed="yes">
+<element name="R4" library="rcl" library_urn="urn:adsk.eagle:library:334" package="M1206" package3d_urn="urn:adsk.eagle:package:23566/2" value="330R" x="25.574" y="24.852" smashed="yes">
 <attribute name="NAME" x="24.304" y="26.122" size="1.27" layer="25"/>
 <attribute name="POPULARITY" value="17" x="72.564" y="-161.838" size="1.778" layer="27" display="off"/>
@@
 <attribute name="VALUE" x="24.304" y="22.312" size="1.27" layer="27"/>
 </element>
-<element name="R5" library="rcl" library_urn="urn:adsk.eagle:library:334" package="M1206" package3d_urn="urn:adsk.eagle:package:23566/2" value="" x="25.186" y="15.68" smashed="yes">
+<element name="R5" library="rcl" library_urn="urn:adsk.eagle:library:334" package="M1206" package3d_urn="urn:adsk.eagle:package:23566/2" value="680R" x="25.186" y="15.68" smashed="yes">
 <attribute name="NAME" x="23.916" y="16.95" size="1.27" layer="25"/>
 <attribute name="POPULARITY" value="17" x="77.256" y="-171.01" size="1.778" layer="27" display="off"/>
@@
 <attribute name="VALUE" x="23.916" y="13.14" size="1.27" layer="27"/>
 </element>
-<element name="R6" library="rcl" library_urn="urn:adsk.eagle:library:334" package="M1206" package3d_urn="urn:adsk.eagle:package:23566/2" value="" x="124.352" y="57.996" smashed="yes" rot="R270">
+<element name="R6" library="rcl" library_urn="urn:adsk.eagle:library:334" package="M1206" package3d_urn="urn:adsk.eagle:package:23566/2" value="330R" x="124.352" y="57.996" smashed="yes" rot="R270">
 <attribute name="NAME" x="125.622" y="59.266" size="1.27" layer="25" rot="R270"/>
 <attribute name="POPULARITY" value="17" x="-62.338" y="0.846" size="1.778" layer="27" rot="R270" display="off"/>
@@
 <attribute name="VALUE" x="121.812" y="59.266" size="1.27" layer="27" rot="R270"/>
 </element>
-<element name="R7" library="rcl" library_urn="urn:adsk.eagle:library:334" package="M1206" package3d_urn="urn:adsk.eagle:package:23566/2" value="" x="127.754" y="55.174" smashed="yes" rot="R270">
+<element name="R7" library="rcl" library_urn="urn:adsk.eagle:library:334" package="M1206" package3d_urn="urn:adsk.eagle:package:23566/2" value="100K" x="127.754" y="55.174" smashed="yes" rot="R270">
 <attribute name="NAME" x="129.024" y="56.444" size="1.27" layer="25" rot="R270"/>
 <attribute name="POPULARITY" value="17" x="-58.936" y="-7.056" size="1.778" layer="27" rot="R270" display="off"/>
@@
 <attribute name="VALUE" x="125.214" y="56.444" size="1.27" layer="27" rot="R270"/>
 </element>
-<element name="R8" library="rcl" library_urn="urn:adsk.eagle:library:334" package="M1206" package3d_urn="urn:adsk.eagle:package:23566/2" value="" x="127.116" y="24.744" smashed="yes" rot="R180">
+<element name="R8" library="rcl" library_urn="urn:adsk.eagle:library:334" package="M1206" package3d_urn="urn:adsk.eagle:package:23566/2" value="100K" x="127.116" y="24.744" smashed="yes" rot="R180">
 <attribute name="NAME" x="128.386" y="23.474" size="1.27" layer="25" rot="R180"/>
 <attribute name="POPULARITY" value="17" x="59.806" y="211.434" size="1.778" layer="27" rot="R180" display="off"/>
@@
 <attribute name="VALUE" x="87.766" y="42.508" size="0.6096" layer="27" font="vector" ratio="20" align="top-center"/>
 </element>
-<element name="F1" library="special" library_urn="urn:adsk.eagle:library:367" package="FUSE1" package3d_urn="urn:adsk.eagle:package:26671/1" value="" x="31.51" y="7.066" smashed="yes" rot="R180">
+<element name="F1" library="special" library_urn="urn:adsk.eagle:library:367" package="FUSE1" package3d_urn="urn:adsk.eagle:package:26671/1" value="1A F" x="31.51" y="7.066" smashed="yes" rot="R180">
 <attribute name="NAME" x="33.415" y="0.081" size="1.778" layer="25" rot="R180"/>
 <attribute name="POPULARITY" value="1" x="31.51" y="7.066" size="1.778" layer="27" rot="R180" display="off"/>
 <attribute name="VALUE" x="33.415" y="2.621" size="1.778" layer="27" rot="R180"/>
 </element>
-<element name="C5" library="rcl" library_urn="urn:adsk.eagle:library:334" package="C1206K" package3d_urn="urn:adsk.eagle:package:23682/2" value="" x="121.488" y="23.102" smashed="yes" rot="R270">
+<element name="C5" library="rcl" library_urn="urn:adsk.eagle:library:334" package="C1206K" package3d_urn="urn:adsk.eagle:package:23682/2" value="100nF" x="121.488" y="23.102" smashed="yes" rot="R270">
 <attribute name="NAME" x="122.588" y="24.702" size="1.016" layer="25" rot="R270"/>
 <attribute name="POPULARITY" value="13" x="121.488" y="23.102" size="1.778" layer="27" rot="R270" display="off"/>
@@
 <attribute name="VALUE" x="119.388" y="24.702" size="1.016" layer="27" rot="R270"/>
 </element>
-<element name="C1" library="rcl" library_urn="urn:adsk.eagle:library:334" package="153CLV-0605" package3d_urn="urn:adsk.eagle:package:23398/2" value="" x="75.594" y="31.1" smashed="yes" rot="MR180">
+<element name="C1" library="rcl" library_urn="urn:adsk.eagle:library:334" package="153CLV-0605" package3d_urn="urn:adsk.eagle:package:23398/2" value="47uF" x="75.594" y="31.1" smashed="yes" rot="MR180">
 <attribute name="NAME" x="72.204" y="27.47" size="1.27" layer="26" rot="MR180"/>
 <attribute name="POPULARITY" value="5" x="66.45" y="19.924" size="1.778" layer="28" rot="MR180" display="off"/>
