File: cad/Eagle/Eagle/Eagle MainPCB/Schulglocke_PCB.brd (EAGLE design)
At the start: 140 x 90 mm, 35 parts, among them M1 DS3231SHIELD, M2 EMC28J60SHIELD, M3 WAVESHAREDISPLAY, Q1 BSS123, Q2 BSS123

Commit message: final version
Parts:
- REL1: device special:REL-5PIN -> customrelay:REL-5PIN
- moved U$3 10.9 mm to (15.2, 57.0)
- moved REL1 1.29 mm to (133.0, 17.0)
- moved M1 0.72 mm to (10.4, 59.9)
- moved R7 0.50 mm to (127.8, 55.2)
Routing:
- net VCC: track 68.3 -> 71.3 mm
- net N$3: track 52.0 -> 53.8 mm
- net N$2: track 48.3 -> 50.2 mm
- net +5V: track 234.0 -> 232.4 mm
- net N$1: track 46.8 -> 48.2 mm
- net ARD_SDA: track 52.5 -> 53.2 mm
- net ARD_SCL: track 52.4 -> 53.1 mm
- net RELAY_EN: track 77.6 -> 78.3 mm
- net N$10: track 10.1 -> 10.8 mm
- added copper zone on layer 1, net GND
- added copper zone on layer 16, net GND
Other:
- board text added: "1"
- board text added: "2"
- board text added: "Michael Schima Viktor Mandlbauer 2022 / 2023"
- board text added: "SV: 2B BV: 1"
- board text added: "Viktor Mandlbauer Michael Schima 2022 / 2023 SV: 2B BV: 1"
