File: cad/Eagle/Eagle/Eagle MainPCB/Schulglocke_PCB.sch (EAGLE design)
At the start: 32 parts, among them M1 DS3231SHIELD, M2 EMC28J60SHIELD, M3 WAVESHAREDISPLAY, Q1 BSS123, Q2 BSS123

Commit message: final version
Parts:
- added U$1, U$2, U$3: MOUNTPOINT3.3MM, customlib:MOUNTPOINT3.3MM
- REL1: device special:REL-5PIN -> customrelay:REL-5PIN
Connections:
- removed net N$18: B2.30
- net RELAY_EN: now also B2.30
Changed lines of the file:
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@@
 <part name="C2" library="rcl" library_urn="urn:adsk.eagle:library:334" deviceset="C-EU" device="102-064X133" package3d_urn="urn:adsk.eagle:package:23653/1"/>
 <part name="C3" library="rcl" library_urn="urn:adsk.eagle:library:334" deviceset="C-EU" device="102-064X133" package3d_urn="urn:adsk.eagle:package:23653/1"/>
-<part name="M1" library="customlib" deviceset="DS3231SHIELD" device=""/>
 <part name="OK1" library="optocoupler" library_urn="urn:adsk.eagle:library:320" deviceset="PC817" device="" package3d_urn="urn:adsk.eagle:package:21938/1"/>
-<part name="REL1" library="special" library_urn="urn:adsk.eagle:library:367" deviceset="REL-5PIN" device="" package3d_urn="urn:adsk.eagle:package:26666/1"/>
 <part name="B2" library="customlib" deviceset="ARDUINO_MEGA_R3_CUSTOM_SHIELD" device="FULL"/>
 <part name="F1" library="special" library_urn="urn:adsk.eagle:library:367" deviceset="FUSE2P" device="" package3d_urn="urn:adsk.eagle:package:26671/1"/>
@@
 <part name="SUPPLY11" library="supply2" library_urn="urn:adsk.eagle:library:372" deviceset="GND" device=""/>
 <part name="C1" library="rcl" library_urn="urn:adsk.eagle:library:334" deviceset="CPOL-EU" device="153CLV-0605" package3d_urn="urn:adsk.eagle:package:23398/2"/>
+<part name="U$1" library="customlib" deviceset="MOUNTPOINT3.3MM" device=""/>
+<part name="U$2" library="customlib" deviceset="MOUNTPOINT3.3MM" device=""/>
+<part name="U$3" library="customlib" deviceset="MOUNTPOINT3.3MM" device=""/>
+<part name="M1" library="customlib" deviceset="DS3231SHIELD" device=""/>
+<part name="REL1" library="customrelay" deviceset="REL-5PIN" device="" package3d_urn="urn:adsk.eagle:package:26666/1"/>
 </parts>
 <sheets>
@@
 <attribute name="VALUE" x="235.204" y="132.461" size="1.778" layer="96"/>
 </instance>
+<instance part="OK1" gate="A" x="129.54" y="152.4" smashed="yes">
+<attribute name="NAME" x="122.555" y="158.115" size="1.778" layer="95"/>
+<attribute name="VALUE" x="122.555" y="144.78" size="1.778" layer="96"/>
+</instance>
+<instance part="B2" gate="B1" x="48.26" y="76.2" smashed="yes">
+<attribute name="NAME" x="35.56" y="132.842" size="1.778" layer="95"/>
+<attribute name="VALUE" x="35.56" y="10.16" size="1.778" layer="96"/>
+</instance>
+<instance part="F1" gate="G$1" x="101.6" y="172.72" smashed="yes">
+<attribute name="NAME" x="100.33" y="174.625" size="1.778" layer="95"/>
+<attribute name="VALUE" x="99.06" y="169.2402" size="1.778" layer="96"/>
+</instance>
+<instance part="C5" gate="G$1" x="165.1" y="162.56" smashed="yes">
+<attribute name="NAME" x="166.624" y="162.941" size="1.778" layer="95"/>
+<attribute name="VALUE" x="166.624" y="157.861" size="1.778" layer="96"/>
+</instance>
+<instance part="P+8" gate="VCC" x="165.1" y="170.18" smashed="yes">
+<attribute name="VALUE" x="162.56" y="167.64" size="1.778" layer="96" rot="R180"/>
+</instance>
+<instance part="SUPPLY11" gate="GND" x="165.1" y="152.4" smashed="yes">
+<attribute name="VALUE" x="163.195" y="149.225" size="1.778" layer="96"/>
+</instance>
+<instance part="C1" gate="G$1" x="172.72" y="162.56" smashed="yes">
+<attribute name="NAME" x="176.403" y="163.0426" size="1.778" layer="95"/>
+<attribute name="VALUE" x="173.863" y="157.9626" size="1.778" layer="96"/>
+</instance>
+<instance part="U$1" gate="G$1" x="12.7" y="68.58" smashed="yes"/>
+<instance part="U$2" gate="G$1" x="12.7" y="83.82" smashed="yes"/>
+<instance part="U$3" gate="G$1" x="12.7" y="53.34" smashed="yes"/>
 <instance part="M1" gate="G$1" x="137.16" y="17.78" smashed="yes">
 <attribute name="NAME" x="127" y="30.48" size="1.778" layer="95"/>
 <attribute name="VALUE" x="127" y="27.94" size="1.778" layer="96"/>
 </instance>
-<instance part="OK1" gate="A" x="129.54" y="152.4" smashed="yes">
-<attribute name="NAME" x="122.555" y="158.115" size="1.778" layer="95"/>
-<attribute name="VALUE" x="122.555" y="144.78" size="1.778" layer="96"/>
-</instance>
 <instance part="REL1" gate="G$1" x="200.66" y="160.02" smashed="yes">
 <attribute name="NAME" x="187.325" y="152.4" size="1.778" layer="95" rot="R90"/>
 <attribute name="VALUE" x="210.82" y="152.4" size="1.778" layer="96" rot="R90"/>
-</instance>
-<instance part="B2" gate="B1" x="48.26" y="76.2" smashed="yes">
-<attribute name="NAME" x="35.56" y="132.842" size="1.778" layer="95"/>
-<attribute name="VALUE" x="35.56" y="10.16" size="1.778" layer="96"/>
-</instance>
-<instance part="F1" gate="G$1" x="101.6" y="172.72" smashed="yes">
-<attribute name="NAME" x="100.33" y="174.625" size="1.778" layer="95"/>
-<attribute name="VALUE" x="99.06" y="169.2402" size="1.778" layer="96"/>
-</instance>
-<instance part="C5" gate="G$1" x="165.1" y="162.56" smashed="yes">
-<attribute name="NAME" x="166.624" y="162.941" size="1.778" layer="95"/>
-<attribute name="VALUE" x="166.624" y="157.861" size="1.778" layer="96"/>
-</instance>
-<instance part="P+8" gate="VCC" x="165.1" y="170.18" smashed="yes">
-<attribute name="VALUE" x="162.56" y="167.64" size="1.778" layer="96" rot="R180"/>
-</instance>
-<instance part="SUPPLY11" gate="GND" x="165.1" y="152.4" smashed="yes">
-<attribute name="VALUE" x="163.195" y="149.225" size="1.778" layer="96"/>
-</instance>
-<instance part="C1" gate="G$1" x="172.72" y="162.56" smashed="yes">
-<attribute name="NAME" x="176.403" y="163.0426" size="1.778" layer="95"/>
-<attribute name="VALUE" x="173.863" y="157.9626" size="1.778" layer="96"/>
 </instance>
 </instances>
@@
 <wire x1="190.5" y1="172.72" x2="190.5" y2="175.26" width="0.1524" layer="91"/>
 <pinref part="D3" gate="1" pin="C"/>
-<pinref part="REL1" gate="G$1" pin="S2"/>
 <wire x1="190.5" y1="170.18" x2="190.5" y2="172.72" width="0.1524" layer="91"/>
 <junction x="190.5" y="172.72"/>
+<pinref part="REL1" gate="G$1" pin="S2"/>
 </segment>
 <segment>
@@
 <wire x1="177.8" y1="147.32" x2="177.8" y2="157.48" width="0.1524" layer="91"/>
 <pinref part="D3" gate="1" pin="A"/>
-<pinref part="REL1" gate="G$1" pin="S1"/>
 <wire x1="190.5" y1="144.78" x2="190.5" y2="147.32" width="0.1524" layer="91"/>
 <pinref part="Q2" gate="G$1" pin="D"/>
@@
 <wire x1="177.8" y1="147.32" x2="190.5" y2="147.32" width="0.1524" layer="91"/>
 <junction x="190.5" y="147.32"/>
+<pinref part="REL1" gate="G$1" pin="S1"/>
 </segment>
 </net>
@@
 <pinref part="JP3" gate="A" pin="2"/>
 <wire x1="220.98" y1="129.54" x2="203.2" y2="129.54" width="0.1524" layer="91"/>
+<wire x1="203.2" y1="129.54" x2="203.2" y2="149.86" width="0.1524" layer="91"/>
 <pinref part="REL1" gate="G$1" pin="C"/>
-<wire x1="203.2" y1="129.54" x2="203.2" y2="149.86" width="0.1524" layer="91"/>
 </segment>
 </net>
@@
 <pinref part="JP3" gate="A" pin="1"/>
 <wire x1="243.84" y1="132.08" x2="254" y2="132.08" width="0.1524" layer="91"/>
-<pinref part="REL1" gate="G$1" pin="O"/>
 <wire x1="208.28" y1="149.86" x2="208.28" y2="144.78" width="0.1524" layer="91"/>
 <wire x1="208.28" y1="144.78" x2="220.98" y2="144.78" width="0.1524" layer="91"/>
 <junction x="220.98" y="144.78"/>
+<pinref part="REL1" gate="G$1" pin="O"/>
 </segment>
 </net>
@@
 <pinref part="JP3" gate="A" pin="3"/>
 <wire x1="243.84" y1="127" x2="254" y2="127" width="0.1524" layer="91"/>
-<pinref part="REL1" gate="G$1" pin="S"/>
 <wire x1="198.12" y1="149.86" x2="198.12" y2="114.3" width="0.1524" layer="91"/>
 <wire x1="198.12" y1="114.3" x2="220.98" y2="114.3" width="0.1524" layer="91"/>
 <junction x="220.98" y="114.3"/>
+<pinref part="REL1" gate="G$1" pin="S"/>
 </segment>
 </net>
@@
 <junction x="152.4" y="137.16"/>
 <label x="137.16" y="137.16" size="1.778" layer="95" rot="R180"/>
+</segment>
+<segment>
+<wire x1="71.12" y1="43.18" x2="63.5" y2="43.18" width="0.1524" layer="91"/>
+<pinref part="B2" gate="B1" pin="30"/>
 <label x="71.12" y="43.18" size="1.778" layer="95"/>
 </segment>
@@
 </segment>
 </net>
-<net name="N$18" class="0">
-<segment>
-<wire x1="71.12" y1="43.18" x2="63.5" y2="43.18" width="0.1524" layer="91"/>
-<pinref part="B2" gate="B1" pin="30"/>
-</segment>
-</net>
